Commit message: Fix Donbot

File: iai_donbot_description/robots/iai_donbot.transmission.xacro (robot description, xacro)
@@ -1,5 +1,6 @@
 <?xml version="1.0"?>
 <robot xmlns:xacro="http://wiki.ros.org/xacro">
-  <xacro:property name="hw_interface" value="hardware_interface/PositionJointInterface" />
+  <xacro:property name="hw_interface" value="hardware_interface/EffortJointInterface" />
+  <xacro:property name="joint_interface" value="EffortJointInterface" />
   <xacro:macro name="ur_arm_transmission" params="prefix">
     <transmission name="${prefix}shoulder_pan_trans">
@@ -9,4 +10,5 @@
       </joint>
       <actuator name="${prefix}shoulder_pan_motor">
+        <hardwareInterface>${joint_interface}</hardwareInterface>
         <mechanicalReduction>1</mechanicalReduction>
       </actuator>
@@ -18,4 +20,5 @@
       </joint>
       <actuator name="${prefix}shoulder_lift_motor">
+        <hardwareInterface>${joint_interface}</hardwareInterface>
         <mechanicalReduction>1</mechanicalReduction>
       </actuator>
@@ -27,4 +30,5 @@
       </joint>
       <actuator name="${prefix}elbow_motor">
+        <hardwareInterface>${joint_interface}</hardwareInterface>
         <mechanicalReduction>1</mechanicalReduction>
       </actuator>
@@ -36,4 +40,5 @@
       </joint>
       <actuator name="${prefix}wrist_1_motor">
+        <hardwareInterface>${joint_interface}</hardwareInterface>
         <mechanicalReduction>1</mechanicalReduction>
       </actuator>
@@ -45,4 +50,5 @@
       </joint>
       <actuator name="${prefix}wrist_2_motor">
+        <hardwareInterface>${joint_interface}</hardwareInterface>
         <mechanicalReduction>1</mechanicalReduction>
       </actuator>
@@ -54,4 +60,25 @@
       </joint>
       <actuator name="${prefix}wrist_3_motor">
+        <hardwareInterface>${joint_interface}</hardwareInterface>
+        <mechanicalReduction>1</mechanicalReduction>
+      </actuator>
+    </transmission>
+    <transmission name="gripper_base_gripper_left_trans">
+      <type>transmission_interface/SimpleTransmission</type>
+      <joint name="gripper_base_gripper_left_joint">
+        <hardwareInterface>${hw_interface}</hardwareInterface>
+      </joint>
+      <actuator name="gripper_base_gripper_left_motor">
+        <hardwareInterface>${joint_interface}</hardwareInterface>
+        <mechanicalReduction>1</mechanicalReduction>
+      </actuator>
+    </transmission>
+    <transmission name="gripper_base_gripper_right_trans">
+      <type>transmission_interface/SimpleTransmission</type>
+      <joint name="gripper_base_gripper_right_joint">
+        <hardwareInterface>${hw_interface}</hardwareInterface>
+      </joint>
+      <actuator name="gripper_base_gripper_right_motor">
+        <hardwareInterface>${joint_interface}</hardwareInterface>
         <mechanicalReduction>1</mechanicalReduction>
       </actuator>

File: iai_donbot_description/robots/iai_donbot.xacro (robot description, xacro)
@@ -1,11 +1,10 @@
 <?xml version="1.0"?>
-<robot xmlns:xacro="http://www.ros.org/wiki/xacro">
-  <xacro:include filename="$(find iai_ur_description)/urdf/common.gazebo.xacro" />
+<robot xmlns:xacro="http://www.ros.org/wiki/xacro" >
   <xacro:include filename="$(find iai_kms_40_description)/urdf/kms_40.urdf.xacro"/>
   <xacro:include filename="$(find iai_adapters_description)/urdf/adapter_fwa050_wsg50.urdf.xacro"/>
   <xacro:include filename="$(find iai_adapters_description)/urdf/adapter_kms40_fwk050.urdf.xacro"/>
   <xacro:include filename="$(find iai_adapters_description)/urdf/fwk_fwa_050.urdf.xacro"/>
-  <xacro:include filename="$(find iai_wsg_50_description)/urdf/wsg_50.urdf.xacro"/>
-  <xacro:include filename="$(find iai_boxy_base_2)/robots/base.URDF.xacro"/>
+  <xacro:include filename="$(find iai_donbot_description)/robots/iai_donbot_gripper.xacro"/>
+  <xacro:include filename="$(find iai_donbot_description)/robots/iai_donbot_base.xacro"/>
   <material name="gray">
     <color rgba="0.56 0.67 0.67 1"/>
@@ -32,8 +31,6 @@
   <xacro:property name="prefix" value="ur5_" />
   <xacro:include filename="$(find iai_ur_description)/urdf/ur5.urdf.xacro" />
-  <xacro:include filename="$(find iai_donbot_description)/robots/iai_donbot.transmission.xacro" /> <!--Override the transmission-->
   <xacro:macro name="iai_donbot">
     <xacro:ur5_robot prefix="${prefix}" joint_limited="false" />
-    <xacro:ur_arm_transmission prefix="${prefix}" />
     <joint name="arm_base_mounting_joint" type="fixed">
       <parent link="base_link" />

File: iai_donbot_description/robots/iai_donbot_spawn.xacro (robot description, xacro)
@@ -2,4 +2,4 @@
 <robot xmlns:xacro="http://www.ros.org/wiki/xacro" name="iai_donbot">
   <xacro:include filename="$(find iai_donbot_description)/robots/iai_donbot.xacro"/>
-  <xacro:iai_donbot/>
+  <xacro:iai_donbot />
 </robot>

File: iai_ur_description/urdf/ur5.urdf.xacro (robot description, xacro)
@@ -1,6 +1,6 @@
 <?xml version="1.0"?>
 <robot xmlns:xacro="http://www.ros.org/wiki/xacro">
-  <xacro:include filename="$(find iai_ur_description)/urdf/ur.transmission.xacro" />
-  <xacro:include filename="$(find iai_ur_description)/urdf/ur.gazebo.xacro" />
+  <!--xacro:include filename="$(find iai_ur_description)/urdf/ur.transmission.xacro" /-->
+  <!--xacro:include filename="$(find iai_ur_description)/urdf/ur.gazebo.xacro" /-->
   <!--xacro:property name="pi" value="3.14159265" /-->
   <!-- Inertia parameters -->
@@ -286,6 +286,6 @@
       </collision>
     </link>
-    <xacro:ur_arm_transmission prefix="${prefix}" />
-    <xacro:ur_arm_gazebo prefix="${prefix}" />
+    <!--xacro:ur_arm_transmission prefix="${prefix}" /-->
+    <!--xacro:ur_arm_gazebo prefix="${prefix}" /-->
     <!-- ROS base_link to UR 'Base' Coordinates transform -->
     <link name="${prefix}base"/>

Commit message: Fix Giskard

File: iai_donbot_description/robots/iai_donbot.transmission.xacro (robot description, xacro)
@@ -1,6 +1,6 @@
 <?xml version="1.0"?>
 <robot xmlns:xacro="http://wiki.ros.org/xacro">
-  <xacro:property name="hw_interface" value="hardware_interface/EffortJointInterface" />
-  <xacro:property name="joint_interface" value="EffortJointInterface" />
+  <xacro:property name="hw_interface" value="hardware_interface/PositionJointInterface" />
+  <xacro:property name="joint_interface" value="PositionJointInterface" />
   <xacro:macro name="ur_arm_transmission" params="prefix">
     <transmission name="${prefix}shoulder_pan_trans">
@@ -10,5 +10,4 @@
       </joint>
       <actuator name="${prefix}shoulder_pan_motor">
-        <hardwareInterface>${joint_interface}</hardwareInterface>
         <mechanicalReduction>1</mechanicalReduction>
       </actuator>
@@ -20,5 +19,4 @@
       </joint>
       <actuator name="${prefix}shoulder_lift_motor">
-        <hardwareInterface>${joint_interface}</hardwareInterface>
         <mechanicalReduction>1</mechanicalReduction>
       </actuator>
@@ -30,5 +28,4 @@
       </joint>
       <actuator name="${prefix}elbow_motor">
-        <hardwareInterface>${joint_interface}</hardwareInterface>
         <mechanicalReduction>1</mechanicalReduction>
       </actuator>
@@ -40,5 +37,4 @@
       </joint>
       <actuator name="${prefix}wrist_1_motor">
-        <hardwareInterface>${joint_interface}</hardwareInterface>
         <mechanicalReduction>1</mechanicalReduction>
       </actuator>
@@ -50,5 +46,4 @@
       </joint>
       <actuator name="${prefix}wrist_2_motor">
-        <hardwareInterface>${joint_interface}</hardwareInterface>
         <mechanicalReduction>1</mechanicalReduction>
       </actuator>
@@ -60,5 +55,4 @@
       </joint>
       <actuator name="${prefix}wrist_3_motor">
-        <hardwareInterface>${joint_interface}</hardwareInterface>
         <mechanicalReduction>1</mechanicalReduction>
       </actuator>
@@ -70,5 +64,4 @@
       </joint>
       <actuator name="gripper_base_gripper_left_motor">
-        <hardwareInterface>${joint_interface}</hardwareInterface>
         <mechanicalReduction>1</mechanicalReduction>
       </actuator>
@@ -80,5 +73,4 @@
       </joint>
       <actuator name="gripper_base_gripper_right_motor">
-        <hardwareInterface>${joint_interface}</hardwareInterface>
         <mechanicalReduction>1</mechanicalReduction>
       </actuator>

Commit message: Fix Control

File: iai_donbot_description/robots/iai_donbot.transmission.xacro (robot description, xacro)
@@ -1,6 +1,5 @@
 <?xml version="1.0"?>
 <robot xmlns:xacro="http://wiki.ros.org/xacro">
-  <xacro:property name="hw_interface" value="hardware_interface/PositionJointInterface" />
-  <xacro:property name="joint_interface" value="PositionJointInterface" />
+  <xacro:property name="hw_interface" value="hardware_interface/EffortJointInterface" />
   <xacro:macro name="ur_arm_transmission" params="prefix">
     <transmission name="${prefix}shoulder_pan_trans">

File: iai_donbot_description/robots/iai_donbot_gazebo.xacro (robot description, xacro)
@@ -5,4 +5,6 @@
     <xacro:include filename="$(find iai_donbot_description)/robots/iai_donbot.transmission.xacro"/>
     <xacro:ur_arm_transmission prefix="ur5_"/>
+    <!-- Load joint controller configurations from YAML file to parameter server -->
+    <rosparam file="$(find iai_donbot_description)/config/iai_donbot_control.yaml" command="load"/>
     <gazebo reference="">
         <plugin name="gazebo_ros_control" filename="libgazebo_ros_control.so">
@@ -11,3 +13,10 @@
         <self_collide>1</self_collide>
     </gazebo>
+    <link name="world">
+    </link>
+    <joint name="world_joint" type="fixed">
+        <origin xyz="0.0 0.0 0.0" rpy="0.0 0.0 0.0"/>
+        <parent link="world"/>
+        <child link="base_link"/>
+    </joint>
 </robot>

Commit message: Add Odom

File: iai_donbot_description/robots/iai_donbot.transmission.xacro (robot description, xacro)
@@ -3,4 +3,31 @@
   <xacro:property name="hw_interface" value="hardware_interface/EffortJointInterface" />
   <xacro:macro name="ur_arm_transmission" params="prefix">
+    <transmission name="odom_x_trans">
+      <type>transmission_interface/SimpleTransmission</type>
+      <joint name="odom_x_joint">
+        <hardwareInterface>${hw_interface}</hardwareInterface>
+      </joint>
+      <actuator name="odom_x_motor">
+        <mechanicalReduction>1</mechanicalReduction>
+      </actuator>
+    </transmission>
+    <transmission name="odom_y_trans">
+      <type>transmission_interface/SimpleTransmission</type>
+      <joint name="odom_y_joint">
+        <hardwareInterface>${hw_interface}</hardwareInterface>
+      </joint>
+      <actuator name="odom_y_motor">
+        <mechanicalReduction>1</mechanicalReduction>
+      </actuator>
+    </transmission>
+    <transmission name="odom_z_trans">
+      <type>transmission_interface/SimpleTransmission</type>
+      <joint name="odom_z_joint">
+        <hardwareInterface>${hw_interface}</hardwareInterface>
+      </joint>
+      <actuator name="odom_z_motor">
+        <mechanicalReduction>1</mechanicalReduction>
+      </actuator>
+    </transmission>
     <transmission name="${prefix}shoulder_pan_trans">
       <type>transmission_interface/SimpleTransmission</type>

File: iai_donbot_description/robots/iai_donbot_base.xacro (robot description, xacro)
@@ -1,3 +1,113 @@
 <robot name="base">
+    <link name="odom">
+        <inertial>
+            <origin xyz="0.0 0.0 0.0" rpy="0.0 0.0 0.0"/>
+            <mass value="1E-4"/>
+            <inertia ixx="1E-4" ixy="0.0" ixz="0.0" iyy="1E-4" iyz="0.0" izz="1E-4"/>
+        </inertial>
+        <visual>
+            <origin rpy="0 0 0" xyz="0 0 0"/>
+            <geometry>
+            <box size="0.01 0.01 0.01"/>
+            </geometry>
+            <material name="White"/>
+        </visual>
+    </link>
+    <joint name="odom_x_joint" type="prismatic">
+        <parent link="odom"/>
+        <child link="odom_x_frame"/>
+        <axis xyz="1 0 0"/>
+        <!-- limits chosen heuristically
+            lower/upper: +-1km to create a quasi limitless prismatic joint
+            velocity: slow walking speed is 3-4km/hour ~= 1m/s
+            effort: reach max speed within 1s, Boxy has a mass of 200kg, so Fmax=200kg*1m/s2 -->
+        <limit lower="-1000" upper="1000" velocity="1" effort="20000"/>
+    </joint>
+    <link name="odom_x_frame">
+        <inertial>
+            <origin xyz="0.0 0.0 0.0" rpy="0.0 0.0 0.0"/>
+            <mass value="1E-4"/>
+            <inertia ixx="1E-4" ixy="0.0" ixz="0.0" iyy="1E-4" iyz="0.0" izz="1E-4"/>
+        </inertial>
+        <visual>
+            <origin rpy="0 0 0" xyz="0 0 0"/>
+            <geometry>
+            <box size="0.01 0.01 0.01"/>
+            </geometry>
+            <material name="White"/>
+        </visual>
+    </link>
+    <joint name="odom_y_joint" type="prismatic">
+        <parent link="odom_x_frame"/>
+        <child link="odom_y_frame"/>
+        <axis xyz="0 1 0"/>
+        <!-- limits chosen heuristically
+            lower/upper: +-1km to create a quasi limitless prismatic joint
+            velocity: slow walking speed is 3-4km/hour ~= 1m/s
+            effort: reach max speed within 1s, Boxy has a mass of 200kg, so Fmax=200kg*1m/s2 -->
+        <limit lower="-1000" upper="1000" velocity="1" effort="20000"/>
+    </joint>
+    <link name="odom_y_frame">
+        <inertial>
+            <origin xyz="0.0 0.0 0.0" rpy="0.0 0.0 0.0"/>
+            <mass value="1E-4"/>
+            <inertia ixx="1E-4" ixy="0.0" ixz="0.0" iyy="1E-4" iyz="0.0" izz="1E-4"/>
+        </inertial>
+        <visual>
+            <origin rpy="0 0 0" xyz="0 0 0"/>
+            <geometry>
+            <box size="0.01 0.01 0.01"/>
+            </geometry>
+            <material name="White"/>
+        </visual>
+    </link>
+    <joint name="odom_z_joint" type="continuous">
+        <parent link="odom_y_frame"/>
+        <child link="base_footprint"/>
+        <axis xyz="0 0 1"/>
+        <!-- limits chosen heuristically
+            velocity: one slow complete turn around in 5-6s, so 6.2rad/6s ~= 1rad/s
+            effort: reach max speed within 1s, Boxy has a mass of 200kg and a diagonale of 1m, so Fmax=200kg*1m*1m/s2 -->
+        <limit velocity="1" effort="20000"/>
+    </joint>
+    <!-- Definition of base_footprint -> base_link -->
+    <link name="base_footprint">
+        <inertial>
+            <origin xyz="0.0 0.0 0.0" rpy="0.0 0.0 0.0"/>
+            <mass value="1E-4"/>
+            <inertia ixx="1E-4" ixy="0.0" ixz="0.0" iyy="1E-4" iyz="0.0" izz="1E-4"/>
+        </inertial>
+        <visual>
+            <origin rpy="0 0 0" xyz="0 0 0"/>
+            <geometry>
+            <box size="0.01 0.01 0.01"/>
+            </geometry>
+            <material name="White"/>
+        </visual>
+    </link>
+    <!-- JOINT to define base_footprint -->
+    <joint name="base_footprint_joint" type="fixed">
+        <!-- Explanation of the calculations to find base_link relative
+        to /base_footprint.
+        /base_footprint is on the floor, exactly in the center of the four wheels to
+        simplify the odometry and FK/IK calculations of the base.
+        Orientation: X pointing forward, and Z up.
+        /base_link is on the front left upper corner of the main alu enclosure.
+            with the same orientation as /base_footprint
+        X:  wheel-axis to wheel-axis distance = 789.5mm.
+            Distance front wheel axis to plane where base_link is: 139.5mm
+            X = 789.5/2 - 139.5 = 255.25mm
+        Y:  main alu enclosure is 450mm wide, and the
+            center of the wheels is also the center of the alu enclosure,
+            so half is Y = 225mm.
+        Z:   base_link is at the top of a 120mm plate.
+            The wheels are aligned with the center of the plate.
+            The wheels are 8", so base_link is
+            Z = 60+4*25.4mm = 161.6mm (above the floor).
+        -->
+        <origin xyz="0.25525 0.225 0.1616" rpy="0 0 0" />
+        <parent link="base_footprint" />
+        <child link="base_link" />
+    </joint>
     <link name="base_link">
         <inertial>

File: iai_donbot_description/robots/iai_donbot_spawn.xacro (robot description, xacro)
@@ -3,3 +3,10 @@
   <xacro:include filename="$(find iai_donbot_description)/robots/iai_donbot.xacro"/>
   <xacro:iai_donbot />
+  <link name="map">
+    </link>
+    <joint name="map_joint" type="fixed">
+        <origin xyz="0.0 0.0 0.0" rpy="0.0 0.0 0.0"/>
+        <parent link="map"/>
+        <child link="odom"/>
+    </joint>
 </robot>

File: iai_donbot_description/robots/iai_donbot_unreal.xacro (robot description, xacro)
@@ -13,9 +13,9 @@
         <self_collide>1</self_collide>
     </gazebo>
-    <link name="world">
+    <link name="map">
     </link>
-    <joint name="world_joint" type="fixed">
+    <joint name="map_joint" type="fixed">
         <origin xyz="0.0 0.0 0.0" rpy="0.0 0.0 0.0"/>
-        <parent link="world"/>
+        <parent link="map"/>
         <child link="odom"/>
     </joint>
